File: stebus-backplane/stebus-backplane.kicad_pcb (KiCad board)
At the start: 4 copper layers, 141.9 x 128.7 mm, 49 parts, among them J101 DIN41612_02x32_AC, J102 DIN41612_02x32_AC, J103 DIN41612_02x32_AC, J104 Soft PWR, J105 ATX-24, J106 DIN41612_02x32_AC, J107 DIN41612_02x32_AC, Q101 2N3904, U101 RT9080

Commit message: multiple in-progress items
Parts:
- removed REF**: OSHW-Logo2_14.6x12mm_SilkScreen, Symbol:OSHW-Logo2_14.6x12mm_SilkScreen
- U101: footprint Package_TO_SOT_SMD:TSOT-23_HandSoldering -> Package_TO_SOT_SMD:SOT-23
- moved U101 0.91 mm to (188.1, 41.1)
Connections:
- U101 pad 1: +5V -> GND
- U101 pad 2: GND -> +2V8
- U101 pad 3: +2V8 -> +5V
Routing:
- net +2V8: track 162.4 -> 165.7 mm
- net +5V: track 3.29 -> 4.36 mm
