File: stebus-backplane/stebus-backplane.kicad_sch (KiCad schematic)
At the start: 48 parts, among them J101 DIN41612_02x32_AC, J102 DIN41612_02x32_AC, J103 DIN41612_02x32_AC, J104 Soft PWR, J105 ATX-24, J106 DIN41612_02x32_AC, J107 DIN41612_02x32_AC, Q101 2N3904, U101 RT9080

Commit message: multiple in-progress items
Parts:
- U101: value RT9080 -> AP2127N-2.8; footprint Package_TO_SOT_SMD:TSOT-23_HandSoldering -> Package_TO_SOT_SMD:SOT-23; symbol vw:RT9080 -> Regulator_Linear:AP2127N-2.8; digikey RT9080-25GJ5 -> 31-AP2127N-2.8TRG1CT-ND
Connections:
- net +2V8: now also U101.2 (VO); no longer U101.3 (VO)
- net +5V: now also U101.3 (VI); no longer U101.1 (VI)
- net GND: now also U101.1 (GND); no longer U101.2 (GND)
Changed lines of the file:
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@@
   (title_block
     (title "5 Slot STEbus Backplane")
-    (date "2023-04-27")
-    (rev "1")
+    (rev "2")
     (company "notcows")
   )
@@
     (stroke (width 0) (type default) (color 0 0 0 0))
   )
-  (wire (pts (xy 133.35 136.525) (xy 129.54 136.525))
+  (wire (pts (xy 135.89 136.525) (xy 129.54 136.525))
     (stroke (width 0) (type default) (color 0 0 0 0))
   )
@@
     (stroke (width 0) (type default) (color 0 0 0 0))
   )
-  (wire (pts (xy 154.94 136.525) (xy 153.67 136.525))
+  (wire (pts (xy 154.94 136.525) (xy 151.13 136.525))
     (stroke (width 0) (type default) (color 0 0 0 0))
   )
@@
     (pin "1")
   )
-  (symbol (lib_id "vw:RT9080") (at 143.51 137.795 0) (mirror y) (unit 1)
+  (symbol (lib_id "Regulator_Linear:AP2127N-2.8") (at 143.51 136.525 0) (mirror y) (unit 1)
     (in_bom yes) (on_board yes) (fields_autoplaced)
-    (property "Reference" "U101" (id 0) (at 143.51 129.413 0))
-    (property "Value" "RT9080" (id 1) (at 143.51 131.953 0))
-    (property "Footprint" "Package_TO_SOT_SMD:TSOT-23_HandSoldering" (id 2) (at 143.51 131.953 0)
-      (effects (font (size 1.27 1.27)) hide)
+    (property "Reference" "U101" (id 0) (at 143.51 128.143 0))
+    (property "Value" "AP2127N-2.8" (id 1) (at 143.51 133.35 0)
+      (effects (font (size 1.27 1.27)) (justify left))
+    )
+    (property "Footprint" "Package_TO_SOT_SMD:SOT-23" (id 2) (at 143.51 130.81 0)
+      (effects (font (size 1.27 1.27) italic) hide)
     )
-    (property "Datasheet" "https://www.richtek.com/SaveDownload.aspx?specid=RT9080" (id 3) (at 143.51 131.953 0)
+    (property "Datasheet" "https://www.diodes.com/assets/Datasheets/AP2127.pdf" (id 3) (at 143.51 136.525 0)
       (effects (font (size 1.27 1.27)) hide)
     )
-    (property "digikey" "RT9080-25GJ5" (id 4) (at 143.51 137.795 0)
+    (property "digikey" "31-AP2127N-2.8TRG1CT-ND" (id 4) (at 143.51 136.525 0)
       (effects (font (size 1.27 1.27)) hide)
     )
@@
     )
     (path "/5de534ff-f627-4c8a-98bf-729c15c69ba6"
-      (reference "U101") (unit 1) (value "RT9080") (footprint "Package_TO_SOT_SMD:TSOT-23_HandSoldering")
+      (reference "U101") (unit 1) (value "AP2127N-2.8") (footprint "Package_TO_SOT_SMD:SOT-23")
     )
   )
